File: kicad/genesis_6button/genesis_6button.sch (KiCad schematic (older format))
At the start: 27 parts, among them J1 Conn_02x07_Odd_Even, J2 DB9_Female, J3 Conn_02x03_Odd_Even, U1 74HC257, U2 ATtiny404-SS, U3 74HC257

Commit message: Revert to first revision of PCB
Parts:
- removed C4: 10u, Capacitor_THT:CP_Radial_D8.0mm_P5.00mm, symbol Device:CP
- removed H1: MountingHole, MountingHole:MountingHole_5.3mm_M5, symbol Mechanical:MountingHole
- removed R13, R14: 100k, Resistor_SMD:R_0805_2012Metric, symbol Device:R
- removed TP1, TP2: TestPoint, TestPoint:TestPoint_Loop_D3.50mm_Drill0.9mm_Beaded, symbol Connector:TestPoint
- C1, C2, C3: footprint Capacitor_SMD:C_1206_3216Metric -> Capacitor_SMD:C_0805_2012Metric
Connections:
- wire segments 129 -> 113
Other:
- moved on the sheet: C2, U2
