File: kicad/genesis_6button/genesis_6button.kicad_pcb (KiCad board)
At the start: 2 copper layers, 74 x 37 mm, 25 parts, among them J1 Conn_02x07_Odd_Even, J2 DB9_Female, J3 Conn_02x03_Odd_Even, U1 74HC257, U2 ATtiny404-SS, U3 74HC257

Commit message: Add gerbers zip file for v1.0
Other:
- rule pad_to_mask_clearance: 0.051 -> 0.05
Changed lines of the file:
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@@
 	)
 	(setup
-		(pad_to_mask_clearance 0.051)
+		(pad_to_mask_clearance 0.05)
 		(allow_soldermask_bridges_in_footprints no)
 		(tenting front back)
@@
 			(usegerberextensions no)
 			(usegerberattributes no)
-			(usegerberadvancedattributes no)
-			(creategerberjobfile no)
+			(usegerberadvancedattributes yes)
+			(creategerberjobfile yes)
 			(dashed_line_dash_ratio 12.000000)
 			(dashed_line_gap_ratio 3.000000)
@@
 			(plotframeref no)
 			(mode 1)
-			(useauxorigin no)
+			(useauxorigin yes)
 			(hpglpennumber 1)
 			(hpglpenspeed 20)
@@
 			(outputformat 1)
 			(mirror no)
-			(drillshape 1)
+			(drillshape 0)
 			(scaleselection 1)
-			(outputdirectory "")
+			(outputdirectory "/home/dan/6button-MD-controller-v1.0-gerbers/")
 		)
 	)
